File: ai03-pcb-guide.kicad_pcb (KiCad board)
At the start: 2 copper layers, 77.8 x 38.1 mm, 24 parts, among them SW1 SW_Push, U1 ATmega32U4-A, Y1 16Mhz

Commit message: Done the guide
Parts:
- moved C1 0.24 mm to (58.2, 73.8)
- renumbered U1 to U2
Connections:
- U2 pad 28: unconnected-(U2-PB4-Pad28) -> ROW0
- U2 pad 29: unconnected-(U2-PB5-Pad29) -> COL1
- U2 pad 30: unconnected-(U2-PB6-Pad30) -> COL0
- U2 pad 31: unconnected-(U2-PC6-Pad31) -> ROW1
Routing:
- net COL1: track 19.0 -> 52.6 mm
- net ROW1: track 21.0 -> 50.8 mm
- net ROW0: track 21.3 -> 49.3 mm
- net COL0: track 19.0 -> 31.9 mm
- net +5V: track 106.6 -> 103.8 mm
- net Net-(U2-UCAP): track 4.16 -> 2.87 mm
- net Net-(U2-D-): track 21.8 -> 22.9 mm, vias 1 -> 2
- net Net-(U2-D+): vias 1 -> 0
- added copper zone on B.Cu, net GND
